Commit message: Updated hexapod geometry with latest version

File: src/hexapod_training/assets/hexapod/hexapod.urdf (robot description, URDF)
Before this commit: robot hexapod, 23 links, 22 joints
Links:
- link base_link: mass 1.0 -> 1.1082; geometry collision box size=0.22 0.161 0.072; visual mesh filename=package://hexapod_description/meshes/body.stl scale=0.001 0.001 0.001
- link camera_link: mass 0.01 -> 0.001
- link front_depth_camera_link: mass 0.02 -> 0.001
- link imu_link: mass 0.01 -> 0.001
- link leg1_coxa: mass 0.1 -> 0.0934
- link leg1_femur: mass 0.05 -> 0.1724
- link leg1_tibia: mass 0.05 -> 0.1034
- link leg2_coxa: mass 0.1 -> 0.0934
- link leg2_femur: mass 0.05 -> 0.1724
- link leg2_tibia: mass 0.05 -> 0.1034
- link leg3_coxa: mass 0.1 -> 0.0934
- link leg3_femur: mass 0.05 -> 0.1724
- link leg3_tibia: mass 0.05 -> 0.1034
- link leg4_coxa: mass 0.1 -> 0.0934
- link leg4_femur: mass 0.05 -> 0.1724
- link leg4_tibia: mass 0.05 -> 0.1034
- link leg5_coxa: mass 0.1 -> 0.0934
- link leg5_femur: mass 0.05 -> 0.1724
- link leg5_tibia: mass 0.05 -> 0.1034
- link leg6_coxa: mass 0.1 -> 0.0934
- link leg6_femur: mass 0.05 -> 0.1724
- link leg6_tibia: mass 0.05 -> 0.1034
- link lidar_link: mass 0.19 -> 0.001
Joints:
- joint leg1_coxa_joint: origin xyz=0.10465180361560904 -0.10465180361560904 0 rpy=0 0 -0.7853981633974483 -> xyz=0.11916 -0.08952 0 rpy=0 0 -0.7853981633974483
- joint leg2_coxa_joint: origin xyz=0 -0.148 0 rpy=0 0 -1.5707963267948966 -> xyz=0 -0.11836 0 rpy=0 0 -1.5707963267948966
- joint leg3_coxa_joint: origin xyz=-0.10465180361560904 -0.10465180361560904 0 rpy=0 0 -2.356194490192345 -> xyz=-0.11916 -0.08952 0 rpy=0 0 -2.356194490192345
- joint leg4_coxa_joint: origin xyz=-0.10465180361560904 0.10465180361560904 0 rpy=0 0 2.356194490192345 -> xyz=-0.11916 0.08952 0 rpy=0 0 2.356194490192345
- joint leg5_coxa_joint: origin xyz=0 0.148 0 rpy=0 0 1.5707963267948966 -> xyz=0 0.11836 0 rpy=0 0 1.5707963267948966
- joint leg6_coxa_joint: origin xyz=0.10465180361560904 0.10465180361560904 0 rpy=0 0 0.7853981633974483 -> xyz=0.11916 0.08952 0 rpy=0 0 0.7853981633974483
